File: NerfPWM.sch (EAGLE design)
At the start: 37 parts, among them IC1 MEGA48/88/168-AU, Q1 MOSFET-NCHANNELSMD, Q2 MOSFET-NCHANNELSMD

Commit message: Changed ISP header.
Parts:
- JP1: value AVR-ISP-6R -> AVR-ISP-6; device custom:AVR-ISP-6R -> custom:AVR-ISP-6
Changed lines of the file:
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@@
 <part name="GND5" library="SparkFun" deviceset="GND" device=""/>
 <part name="GND6" library="SparkFun" deviceset="GND" device=""/>
-<part name="JP1" library="custom" deviceset="AVR-ISP-6" device="R" value="AVR-ISP-6R"/>
+<part name="JP1" library="custom" deviceset="AVR-ISP-6" device="" value="AVR-ISP-6"/>
 <part name="U$6" library="SparkFun" deviceset="5V" device=""/>
 <part name="GND7" library="SparkFun" deviceset="GND" device=""/>
