File: NerfPWM.brd (EAGLE design)
At the start: 50.8 x 25.4 mm, 37 parts, among them IC1 MEGA48/88/168-AU

Commit message: Increased spacing around FET ground connections.
Connections:
- new net N$1: IC1.20
Changed lines of the file:
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@@
 <vertex x="27.305" y="12.065"/>
 </polygon>
-<polygon width="0.3048" layer="1" thermals="no">
+<polygon width="0.3048" layer="1" isolate="0.3048" thermals="no">
 <vertex x="35.56" y="5.08"/>
 <vertex x="33.02" y="5.08"/>
@@
 <vertex x="35.56" y="8.89"/>
 </polygon>
-<polygon width="0.3048" layer="1" thermals="no">
+<polygon width="0.3048" layer="1" isolate="0.3048" thermals="no">
 <vertex x="31.75" y="24.13"/>
 <vertex x="31.75" y="24.765"/>
@@
 <wire x1="10.0584" y1="2.286" x2="9.144" y2="2.286" width="0.1524" layer="16"/>
 </signal>
+<signal name="N$1">
+<contactref element="IC1" pad="20"/>
+</signal>
 </signals>
