File: NerfPWM.brd (EAGLE design)
At the start: 50.8 x 25.4 mm, 37 parts, among them IC1 MEGA48/88/168-AU

Commit message: Board revisions for easier assembly of next batch.
Parts:
- moved PBRAKE1 4.07 mm to (33.7, 17.8)
- moved PBRAKE2 3.86 mm to (28.2, 1.24)
- moved PWM2 2.29 mm to (29.5, 8.56)
- moved R1 2.29 mm to (30.5, 6.99), turned to 0 degrees
- moved PWM1 2.01 mm to (28.6, 21.9)
- moved BRAKE2 1.91 mm to (27.4, 6.99)
- moved R2 1.81 mm to (31.1, 1.27), turned to 0 degrees
- moved Q2 1.78 mm to (30.6, 4.14)
- moved R5 1.61 mm to (30.8, 20.7), turned to 0 degrees
- moved R3 1.60 mm to (27.3, 4.14)
- moved R4 1.54 mm to (30.9, 23.7), turned to 0 degrees
- moved Q1 0.63 mm to (31.1, 17.8)
Routing:
- net N$3: track 6.42 -> 8.17 mm
- net PWM2: track 16.6 -> 18.1 mm
- net N$2: track 7.22 -> 8.70 mm
- net +12V: track 4.18 -> 2.85 mm
- net GND: track 14.8 -> 15.9 mm
- net PWM1: track 21.2 -> 22.3 mm
- net BRAKE1: track 39.1 -> 39.7 mm
- net BRAKE2: track 24.7 -> 24.1 mm
Other:
- board text added: "NerfPWM V1.2 2013-??-?? Thomas Deal"
- board text removed: "NerfPWM V1.1 2013-09-27 Thomas Deal"
